File: shema/ultrasonicsensor3.sch (EAGLE design)
At the start: 22 parts, among them IC1 PIC12F675P, T1 DAP 202 UM

Commit message: shema
Parts:
- removed R1: 1k, rcl:R-EU_0207/2V
- added F1: (no value), fuse:SH22,5A
Connections:
- new net N$9: F1.1
- net 220-1: now also F1.2
- net DOOR: no longer R1.2
- net N$5: no longer R1.1
Other:
- note added: "Travel Charger Nokia AC-2E Input: ~ 100-240V/150mA Output: 5.3V/500mA"
- note removed: "Travel Charger In: 110/220V Out: 5V"
Changed lines of the file:
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@@
 <layer number="56" name="wert" color="7" fill="1" visible="no" active="no"/>
 <layer number="57" name="tCAD" color="7" fill="1" visible="no" active="no"/>
+<layer number="90" name="Modules" color="5" fill="1" visible="yes" active="yes"/>
 <layer number="91" name="Nets" color="2" fill="1" visible="yes" active="yes"/>
 <layer number="92" name="Busses" color="1" fill="1" visible="yes" active="yes"/>
@@
 </class>
 </classes>
+<modules>
+<module name="1" prefix="" dx="30.48" dy="15.24">
+<ports>
+</ports>
+<variantdefs>
+</variantdefs>
+<parts>
+</parts>
+<sheets>
+<sheet>
+<plain>
+</plain>
+<instances>
+</instances>
+<busses>
+</busses>
+<nets>
+</nets>
+</sheet>
+</sheets>
+</module>
+</modules>
 <parts>
 <part name="IC1" library="microchip" deviceset="PIC12F675" device="P"/>
@@
 <part name="GND15" library="supply1" deviceset="GND" device=""/>
 <part name="GND10" library="supply1" deviceset="GND" device=""/>
-<part name="R1" library="rcl" deviceset="R-EU_" device="0207/2V" value="1k"/>
 <part name="LED1" library="led" deviceset="LED" device="3MM"/>
 <part name="LED2" library="led" deviceset="LED" device="3MM"/>
@@
 <part name="C1" library="rcl" deviceset="CPOL-EU" device="C/6032-28R" value="50x10V"/>
 <part name="GND4" library="supply1" deviceset="GND" device=""/>
+<part name="F1" library="fuse" deviceset="SH22,5A" device=""/>
 </parts>
 <sheets>
@@
 <text x="106.68" y="177.8" size="1.778" layer="91">220V LOAD</text>
 <text x="106.68" y="185.42" size="1.778" layer="91">220V IN</text>
-<text x="7.62" y="175.26" size="1.778" layer="91">Travel Charger
-In:   110/220V
-Out: 5V</text>
-<text x="-2.54" y="180.34" size="1.778" layer="91">6V</text>
+<text x="3.302" y="172.974" size="1.778" layer="91">Travel Charger
+Nokia AC-2E
+Input:  ~ 100-240V/150mA
+Output: 5.3V/500mA</text>
+<text x="-2.794" y="181.102" size="1.778" layer="91">6V</text>
 </plain>
+<moduleinsts>
+<moduleinst name="." module="1" x="17.78" y="177.8"/>
+</moduleinsts>
 <instances>
 <instance part="IC1" gate="G$1" x="17.78" y="121.92"/>
@@
 <attribute name="VALUE" x="0" y="170.18" size="1.778" layer="96" rot="MR0"/>
 </instance>
-<instance part="R1" gate="G$1" x="48.26" y="121.92"/>
 <instance part="LED1" gate="G$1" x="50.8" y="139.7" rot="R90"/>
 <instance part="LED2" gate="G$1" x="0" y="162.56" rot="R90"/>
@@
 </instance>
 <instance part="GND4" gate="1" x="17.78" y="144.78" rot="MR0"/>
+<instance part="F1" gate="1" x="53.34" y="180.34"/>
 </instances>
 <busses>
@@
 </segment>
 <segment>
-<wire x1="2.54" y1="175.26" x2="2.54" y2="172.72" width="0.1524" layer="91"/>
-<wire x1="2.54" y1="172.72" x2="2.54" y2="170.18" width="0.1524" layer="91"/>
-<wire x1="2.54" y1="170.18" x2="27.94" y2="170.18" width="0.1524" layer="91"/>
-<wire x1="27.94" y1="170.18" x2="27.94" y2="185.42" width="0.1524" layer="91"/>
-<wire x1="27.94" y1="185.42" x2="2.54" y2="185.42" width="0.1524" layer="91"/>
-<wire x1="2.54" y1="185.42" x2="2.54" y2="180.34" width="0.1524" layer="91"/>
-<wire x1="2.54" y1="180.34" x2="2.54" y2="175.26" width="0.1524" layer="91"/>
-<wire x1="2.54" y1="180.34" x2="2.54" y2="175.26" width="0.1524" layer="91"/>
-<wire x1="2.54" y1="175.26" x2="2.54" y2="172.72" width="0.1524" layer="91"/>
 <wire x1="2.54" y1="175.26" x2="-2.54" y2="175.26" width="0.1524" layer="91"/>
 <pinref part="GND10" gate="1" pin="GND"/>
@@
 <wire x1="86.36" y1="182.88" x2="101.6" y2="182.88" width="0.1524" layer="91"/>
 <wire x1="86.36" y1="182.88" x2="83.82" y2="182.88" width="0.1524" layer="91"/>
-<wire x1="83.82" y1="182.88" x2="53.34" y2="182.88" width="0.1524" layer="91"/>
-<wire x1="53.34" y1="182.88" x2="53.34" y2="175.26" width="0.1524" layer="91"/>
-<wire x1="53.34" y1="175.26" x2="27.94" y2="175.26" width="0.1524" layer="91"/>
+<wire x1="83.82" y1="182.88" x2="68.58" y2="182.88" width="0.1524" layer="91"/>
+<wire x1="68.58" y1="182.88" x2="68.58" y2="175.26" width="0.1524" layer="91"/>
+<wire x1="68.58" y1="175.26" x2="33.02" y2="175.26" width="0.1524" layer="91"/>
 <pinref part="RL1" gate="K1" pin="6"/>
 <wire x1="83.82" y1="162.56" x2="83.82" y2="182.88" width="0.1524" layer="91"/>
@@
 <pinref part="JP2" gate="G$3" pin="1"/>
 <wire x1="101.6" y1="185.42" x2="96.52" y2="185.42" width="0.1524" layer="91"/>
-<wire x1="96.52" y1="185.42" x2="48.26" y2="185.42" width="0.1524" layer="91"/>
+<wire x1="96.52" y1="185.42" x2="66.04" y2="185.42" width="0.1524" layer="91"/>
 <pinref part="JP2" gate="G$3" pin="4"/>
 <wire x1="101.6" y1="177.8" x2="96.52" y2="177.8" width="0.1524" layer="91"/>
 <wire x1="96.52" y1="177.8" x2="96.52" y2="185.42" width="0.1524" layer="91"/>
 <junction x="96.52" y="185.42"/>
-<wire x1="48.26" y1="185.42" x2="48.26" y2="180.34" width="0.1524" layer="91"/>
-<wire x1="48.26" y1="180.34" x2="27.94" y2="180.34" width="0.1524" layer="91"/>
+<wire x1="66.04" y1="185.42" x2="66.04" y2="180.34" width="0.1524" layer="91"/>
+<pinref part="F1" gate="1" pin="2"/>
+<wire x1="58.42" y1="180.34" x2="66.04" y2="180.34" width="0.1524" layer="91"/>
 </segment>
 </net>
@@
 </segment>
 <segment>
-<wire x1="53.34" y1="121.92" x2="55.88" y2="121.92" width="0.1524" layer="91"/>
-<label x="55.88" y="121.92" size="1.778" layer="95" xref="yes"/>
-<pinref part="R1" gate="G$1" pin="2"/>
+<wire x1="43.18" y1="121.92" x2="48.26" y2="121.92" width="0.1524" layer="91"/>
+<label x="48.26" y="121.92" size="1.778" layer="95" xref="yes"/>
 </segment>
 </net>
@@
 <pinref part="IC1" gate="G$1" pin="GP2/AN2"/>
 <wire x1="33.02" y1="121.92" x2="43.18" y2="121.92" width="0.1524" layer="91"/>
-<pinref part="R1" gate="G$1" pin="1"/>
 </segment>
 </net>
@@
 </segment>
 </net>
+<net name="N$9" class="0">
+<segment>
+<pinref part="F1" gate="1" pin="1"/>
+<wire x1="48.26" y1="180.34" x2="33.02" y2="180.34" width="0.1524" layer="91"/>
+</segment>
+</net>
