File: shema/ultrasonicsensor4.sch (EAGLE design)
At the start: 27 parts, among them IC1 PIC12F675P, T1 DAP 202 UM

Commit message: modified:   ultrasonicsensor4.sch
Connections:
- removed net N$4: C9.2, JP3.1, R3.2, USONIC.5V
- new net ECHO: IC1.GP3/!MCLR, JP4.3
- new net N$12: C9.2, JP3.1, USONIC.5V
- net GND: now also R3.2
- net TRIG: now also JP4.2
- net VPP: no longer IC1.GP3/!MCLR
Other:
- moved on the sheet: R3
Changed lines of the file:
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@@
 <instance part="S2" gate="-LED" x="147.32" y="152.4"/>
 <instance part="R1" gate="G$1" x="147.32" y="142.24" rot="R270"/>
-<instance part="R3" gate="G$1" x="172.72" y="142.24" rot="R270"/>
+<instance part="R3" gate="G$1" x="154.94" y="142.24" rot="R270"/>
 <instance part="GND5" gate="1" x="119.38" y="119.38" rot="R180"/>
 </instances>
@@
 <net name="TRIG" class="0">
 <segment>
-<wire x1="0" y1="93.98" x2="-5.08" y2="93.98" width="0.1524" layer="91"/>
+<wire x1="5.08" y1="101.6" x2="-5.08" y2="101.6" width="0.1524" layer="91"/>
 <pinref part="IC1" gate="G$1" pin="GP5/CLKIN"/>
-<wire x1="-5.08" y1="93.98" x2="-5.08" y2="116.84" width="0.1524" layer="91"/>
+<wire x1="-5.08" y1="101.6" x2="-5.08" y2="116.84" width="0.1524" layer="91"/>
 <wire x1="-5.08" y1="116.84" x2="5.08" y2="116.84" width="0.1524" layer="91"/>
-<label x="0" y="93.98" size="1.778" layer="95" xref="yes"/>
+<label x="5.08" y="101.6" size="1.778" layer="95" xref="yes"/>
 </segment>
 <segment>
@@
 <label x="137.16" y="127" size="1.778" layer="95" rot="R90"/>
 </segment>
+<segment>
+<pinref part="JP4" gate="G$3" pin="2"/>
+<wire x1="101.6" y1="106.68" x2="86.36" y2="106.68" width="0.1524" layer="91"/>
+<label x="86.36" y="106.68" size="1.778" layer="95" rot="R180" xref="yes"/>
+</segment>
 </net>
 <net name="GND" class="0">
@@
 <junction x="147.32" y="116.84"/>
 <pinref part="R1" gate="G$1" pin="2"/>
-<wire x1="147.32" y1="137.16" x2="147.32" y2="116.84" width="0.1524" layer="91"/>
+<wire x1="147.32" y1="137.16" x2="147.32" y2="129.54" width="0.1524" layer="91"/>
 <pinref part="GND5" gate="1" pin="GND"/>
+<wire x1="147.32" y1="129.54" x2="147.32" y2="116.84" width="0.1524" layer="91"/>
 <wire x1="119.38" y1="116.84" x2="119.38" y2="111.76" width="0.1524" layer="91"/>
 <junction x="119.38" y="111.76"/>
+<pinref part="R3" gate="G$1" pin="2"/>
+<wire x1="154.94" y1="137.16" x2="154.94" y2="129.54" width="0.1524" layer="91"/>
+<wire x1="154.94" y1="129.54" x2="147.32" y2="129.54" width="0.1524" layer="91"/>
+<junction x="147.32" y="129.54"/>
 </segment>
 </net>
@@
 <wire x1="-10.16" y1="101.6" x2="-10.16" y2="114.3" width="0.1524" layer="91"/>
 <label x="-10.16" y="106.68" size="1.778" layer="95" rot="R90"/>
-</segment>
-<segment>
-<pinref part="IC1" gate="G$1" pin="GP3/!MCLR"/>
-<wire x1="5.08" y1="129.54" x2="-5.08" y2="129.54" width="0.1524" layer="91"/>
-<label x="-5.08" y="127.508" size="1.778" layer="95"/>
 </segment>
 </net>
@@
 </segment>
 </net>
-<net name="N$4" class="0">
-<segment>
-<pinref part="JP3" gate="G$3" pin="1"/>
-<wire x1="114.3" y1="104.14" x2="142.24" y2="104.14" width="0.1524" layer="91"/>
-<wire x1="142.24" y1="104.14" x2="142.24" y2="101.6" width="0.1524" layer="91"/>
-<pinref part="USONIC" gate="J_ULTRASONIC" pin="5V"/>
-<wire x1="142.24" y1="101.6" x2="147.32" y2="101.6" width="0.1524" layer="91"/>
-<pinref part="C9" gate="G$1" pin="2"/>
-<wire x1="147.32" y1="101.6" x2="152.4" y2="101.6" width="0.1524" layer="91"/>
-<wire x1="152.4" y1="101.6" x2="154.94" y2="101.6" width="0.1524" layer="91"/>
-<wire x1="147.32" y1="99.06" x2="147.32" y2="101.6" width="0.1524" layer="91"/>
-<junction x="147.32" y="101.6"/>
-<pinref part="R3" gate="G$1" pin="2"/>
-<wire x1="172.72" y1="137.16" x2="172.72" y2="91.44" width="0.1524" layer="91"/>
-<wire x1="172.72" y1="91.44" x2="152.4" y2="91.44" width="0.1524" layer="91"/>
-<wire x1="152.4" y1="91.44" x2="152.4" y2="101.6" width="0.1524" layer="91"/>
-<junction x="152.4" y="101.6"/>
-</segment>
-</net>
 <net name="N$13" class="0">
 <segment>
@@
 <segment>
 <pinref part="R3" gate="G$1" pin="1"/>
-<wire x1="172.72" y1="165.1" x2="172.72" y2="147.32" width="0.1524" layer="91"/>
+<wire x1="154.94" y1="165.1" x2="154.94" y2="147.32" width="0.1524" layer="91"/>
 <pinref part="S2" gate="-1" pin="1A"/>
-<wire x1="172.72" y1="165.1" x2="152.4" y2="165.1" width="0.1524" layer="91"/>
-</segment>
-</net>
+<wire x1="154.94" y1="165.1" x2="152.4" y2="165.1" width="0.1524" layer="91"/>
+</segment>
+</net>
+<net name="ECHO" class="0">
+<segment>
+<pinref part="IC1" gate="G$1" pin="GP3/!MCLR"/>
+<wire x1="5.08" y1="129.54" x2="-5.08" y2="129.54" width="0.1524" layer="91"/>
+<label x="-5.08" y="129.54" size="1.778" layer="95" rot="R180" xref="yes"/>
+</segment>
+<segment>
+<pinref part="JP4" gate="G$3" pin="3"/>
+<wire x1="101.6" y1="109.22" x2="96.52" y2="109.22" width="0.1524" layer="91"/>
+<label x="96.52" y="109.22" size="1.778" layer="95" rot="R180" xref="yes"/>
+</segment>
+</net>
+<net name="N$12" class="0">
+<segment>
+<pinref part="USONIC" gate="J_ULTRASONIC" pin="5V"/>
+<pinref part="JP3" gate="G$3" pin="1"/>
+<wire x1="114.3" y1="104.14" x2="142.24" y2="104.14" width="0.1524" layer="91"/>
+<wire x1="142.24" y1="104.14" x2="142.24" y2="101.6" width="0.1524" layer="91"/>
+<wire x1="142.24" y1="101.6" x2="147.32" y2="101.6" width="0.1524" layer="91"/>
+<pinref part="C9" gate="G$1" pin="2"/>
+<wire x1="147.32" y1="99.06" x2="147.32" y2="101.6" width="0.1524" layer="91"/>
+<junction x="147.32" y="101.6"/>
+<wire x1="147.32" y1="101.6" x2="154.94" y2="101.6" width="0.1524" layer="91"/>
+</segment>
+</net>

Commit message: shema. added BUZZER
Parts:
- added Q3: AP70T03GH, adafruit:MOSFET-NREFLOW
- added SG1: KPX-G1212B, buzzer:EB2505
Connections:
- new net BUZZER: Q3.G
- new net N$4: Q3.D, SG1.-
- net GND: now also Q3.S
- net N$1: now also SG1.+
Other:
- moved on the sheet: R1, R3, S2-1, S2-LED
Changed lines of the file:
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@@
 <part name="R3" library="rcl" deviceset="R-EU_" device="0207/2V" value="1k"/>
 <part name="GND5" library="supply1" deviceset="GND" device=""/>
+<part name="SG1" library="buzzer" deviceset="EB2505" device="" value="KPX-G1212B"/>
+<part name="Q3" library="adafruit" deviceset="MOSFET-N" device="REFLOW" value="AP70T03GH"/>
+<part name="GND6" library="supply1" deviceset="GND" device=""/>
 </parts>
 <sheets>
@@
 <instance part="JP4" gate="G$3" x="104.14" y="104.14" rot="MR90"/>
 <instance part="GND2" gate="1" x="96.52" y="119.38" rot="R180"/>
-<instance part="S2" gate="-1" x="147.32" y="165.1" rot="MR0"/>
-<instance part="S2" gate="-LED" x="147.32" y="152.4"/>
-<instance part="R1" gate="G$1" x="147.32" y="142.24" rot="R270"/>
-<instance part="R3" gate="G$1" x="154.94" y="142.24" rot="R270"/>
+<instance part="S2" gate="-1" x="147.32" y="154.94" rot="MR0"/>
+<instance part="S2" gate="-LED" x="147.32" y="142.24"/>
+<instance part="R1" gate="G$1" x="147.32" y="129.54" rot="R270"/>
+<instance part="R3" gate="G$1" x="154.94" y="129.54" rot="R270"/>
 <instance part="GND5" gate="1" x="119.38" y="119.38" rot="R180"/>
+<instance part="SG1" gate="G$1" x="-17.78" y="147.32" smashed="yes" rot="R270">
+<attribute name="NAME" x="-11.43" y="149.86" size="1.778" layer="95" rot="R270"/>
+<attribute name="VALUE" x="-7.366" y="140.716" size="1.778" layer="96" rot="R90"/>
+</instance>
+<instance part="Q3" gate="G$1" x="-22.86" y="137.16"/>
+<instance part="GND6" gate="1" x="-20.32" y="127" rot="MR0"/>
 </instances>
 <busses>
@@
 <wire x1="114.3" y1="106.68" x2="137.16" y2="106.68" width="0.1524" layer="91"/>
 <wire x1="137.16" y1="106.68" x2="154.94" y2="106.68" width="0.1524" layer="91"/>
-<wire x1="137.16" y1="162.56" x2="137.16" y2="157.48" width="0.1524" layer="91"/>
+<wire x1="137.16" y1="152.4" x2="137.16" y2="147.32" width="0.1524" layer="91"/>
 <junction x="137.16" y="106.68"/>
 <pinref part="S2" gate="-1" pin="NO"/>
-<wire x1="137.16" y1="157.48" x2="137.16" y2="106.68" width="0.1524" layer="91"/>
-<wire x1="137.16" y1="162.56" x2="142.24" y2="162.56" width="0.1524" layer="91"/>
+<wire x1="137.16" y1="147.32" x2="137.16" y2="106.68" width="0.1524" layer="91"/>
+<wire x1="137.16" y1="152.4" x2="142.24" y2="152.4" width="0.1524" layer="91"/>
 <pinref part="S2" gate="-LED" pin="A"/>
-<wire x1="147.32" y1="154.94" x2="147.32" y2="157.48" width="0.1524" layer="91"/>
-<wire x1="147.32" y1="157.48" x2="137.16" y2="157.48" width="0.1524" layer="91"/>
-<junction x="137.16" y="157.48"/>
+<wire x1="147.32" y1="144.78" x2="147.32" y2="147.32" width="0.1524" layer="91"/>
+<wire x1="147.32" y1="147.32" x2="137.16" y2="147.32" width="0.1524" layer="91"/>
+<junction x="137.16" y="147.32"/>
 <label x="137.16" y="127" size="1.778" layer="95" rot="R90"/>
 </segment>
@@
 <junction x="147.32" y="116.84"/>
 <pinref part="R1" gate="G$1" pin="2"/>
-<wire x1="147.32" y1="137.16" x2="147.32" y2="129.54" width="0.1524" layer="91"/>
+<wire x1="147.32" y1="124.46" x2="147.32" y2="121.92" width="0.1524" layer="91"/>
 <pinref part="GND5" gate="1" pin="GND"/>
-<wire x1="147.32" y1="129.54" x2="147.32" y2="116.84" width="0.1524" layer="91"/>
+<wire x1="147.32" y1="121.92" x2="147.32" y2="116.84" width="0.1524" layer="91"/>
 <wire x1="119.38" y1="116.84" x2="119.38" y2="111.76" width="0.1524" layer="91"/>
 <junction x="119.38" y="111.76"/>
 <pinref part="R3" gate="G$1" pin="2"/>
-<wire x1="154.94" y1="137.16" x2="154.94" y2="129.54" width="0.1524" layer="91"/>
-<wire x1="154.94" y1="129.54" x2="147.32" y2="129.54" width="0.1524" layer="91"/>
-<junction x="147.32" y="129.54"/>
+<wire x1="154.94" y1="124.46" x2="154.94" y2="121.92" width="0.1524" layer="91"/>
+<wire x1="154.94" y1="121.92" x2="147.32" y2="121.92" width="0.1524" layer="91"/>
+<junction x="147.32" y="121.92"/>
+</segment>
+<segment>
+<pinref part="Q3" gate="G$1" pin="S"/>
+<pinref part="GND6" gate="1" pin="GND"/>
+<wire x1="-20.32" y1="132.08" x2="-20.32" y2="129.54" width="0.1524" layer="91"/>
 </segment>
 </net>
@@
 </segment>
 </net>
-<net name="TX-RS232" class="0">
+<net name="BUZZER" class="0">
 <segment>
 <wire x1="35.56" y1="134.62" x2="38.1" y2="134.62" width="0.1524" layer="91"/>
 <label x="38.1" y="134.62" size="1.778" layer="95" rot="R90" xref="yes"/>
+</segment>
+<segment>
+<pinref part="Q3" gate="G$1" pin="G"/>
+<wire x1="-25.4" y1="134.62" x2="-27.94" y2="134.62" width="0.1524" layer="91"/>
+<label x="-27.94" y="134.62" size="1.778" layer="95" rot="R90" xref="yes"/>
 </segment>
 </net>
@@
 <wire x1="71.12" y1="167.64" x2="71.12" y2="163.83" width="0.1524" layer="91"/>
 <junction x="71.12" y="167.64"/>
-<wire x1="-15.24" y1="157.48" x2="-7.62" y2="157.48" width="0.1524" layer="91"/>
-<wire x1="-15.24" y1="157.48" x2="-25.4" y2="157.48" width="0.1524" layer="91"/>
-<wire x1="-25.4" y1="167.64" x2="-25.4" y2="157.48" width="0.1524" layer="91"/>
-<wire x1="53.34" y1="167.64" x2="-25.4" y2="167.64" width="0.1524" layer="91"/>
+<wire x1="-5.08" y1="157.48" x2="-20.32" y2="157.48" width="0.1524" layer="91"/>
+<wire x1="-20.32" y1="167.64" x2="-20.32" y2="157.48" width="0.1524" layer="91"/>
+<wire x1="53.34" y1="167.64" x2="-20.32" y2="167.64" width="0.1524" layer="91"/>
 <junction x="53.34" y="167.64"/>
-<wire x1="-25.4" y1="167.64" x2="-25.4" y2="180.34" width="0.1524" layer="91"/>
-<junction x="-25.4" y="167.64"/>
-<wire x1="-25.4" y1="180.34" x2="-5.08" y2="180.34" width="0.1524" layer="91"/>
-<wire x1="-5.08" y1="180.34" x2="2.286" y2="180.34" width="0.1524" layer="91"/>
+<wire x1="-20.32" y1="167.64" x2="-20.32" y2="180.34" width="0.1524" layer="91"/>
+<junction x="-20.32" y="167.64"/>
+<wire x1="-20.32" y1="180.34" x2="2.286" y2="180.34" width="0.1524" layer="91"/>
 <pinref part="LED2" gate="G$1" pin="A"/>
 <wire x1="-2.54" y1="162.56" x2="-5.08" y2="162.56" width="0.1524" layer="91"/>
@@
 <wire x1="-5.08" y1="157.48" x2="-5.08" y2="152.4" width="0.1524" layer="91"/>
 <wire x1="-5.08" y1="152.4" x2="-2.54" y2="152.4" width="0.1524" layer="91"/>
-<wire x1="-7.62" y1="157.48" x2="-5.08" y2="157.48" width="0.1524" layer="91"/>
 <junction x="-5.08" y="157.48"/>
+<pinref part="SG1" gate="G$1" pin="+"/>
+<wire x1="-20.32" y1="149.86" x2="-20.32" y2="157.48" width="0.1524" layer="91"/>
+<junction x="-20.32" y="157.48"/>
 </segment>
 </net>
@@
 <pinref part="S2" gate="-LED" pin="K"/>
 <pinref part="R1" gate="G$1" pin="1"/>
+<wire x1="147.32" y1="134.62" x2="147.32" y2="137.16" width="0.1524" layer="91"/>
 </segment>
 </net>
@@
 <segment>
 <pinref part="R3" gate="G$1" pin="1"/>
-<wire x1="154.94" y1="165.1" x2="154.94" y2="147.32" width="0.1524" layer="91"/>
+<wire x1="154.94" y1="154.94" x2="154.94" y2="134.62" width="0.1524" layer="91"/>
 <pinref part="S2" gate="-1" pin="1A"/>
-<wire x1="154.94" y1="165.1" x2="152.4" y2="165.1" width="0.1524" layer="91"/>
+<wire x1="154.94" y1="154.94" x2="152.4" y2="154.94" width="0.1524" layer="91"/>
 </segment>
 </net>
@@
 </segment>
 </net>
+<net name="N$4" class="0">
+<segment>
+<pinref part="SG1" gate="G$1" pin="-"/>
+<pinref part="Q3" gate="G$1" pin="D"/>
+</segment>
+</net>
